Commit message: Adds calibration position

File: kmriiwa_moveit/config/kmriiwa.srdf.xacro (robot description, xacro)
@@ -36,4 +36,14 @@
         <joint name="$(arg robot_name)_joint_6" value="0.8827"/>
         <joint name="$(arg robot_name)_joint_7" value="0.662003"/>
+    </group_state>
+    <!-- Add calibration joint state for each robot -->
+    <group_state name="vicon_calibration" group="$(arg robot_name)_manipulator">
+        <joint name="$(arg robot_name)_joint_1" value="0.7549"/>
+        <joint name="$(arg robot_name)_joint_2" value="-1.3888"/>
+        <joint name="$(arg robot_name)_joint_3" value="-2.0210"/>
+        <joint name="$(arg robot_name)_joint_4" value="-1.9374"/>
+        <joint name="$(arg robot_name)_joint_5" value="-1.5525"/>
+        <joint name="$(arg robot_name)_joint_6" value="-2.0524"/>
+        <joint name="$(arg robot_name)_joint_7" value="2.0660"/>
     </group_state>
     <xacro:unless value="$(arg no_virtual_joint)">
